Commit message: create ros2_package

File: urdf/cirtesub.urdf (robot description, URDF)
Before this commit: robot cirtesub, 9 links, 8 joints
Links:
- link cirtesub/base_link: geometry visual mesh filename=package://cirtesub_description/meshes/cirtesubdae.dae scale=1 1 1

Commit message: moveit configs y diagnostics y ajustes de urdf para general integration de sura

File: urdf/cirtesub.urdf (robot description, URDF)
Before this commit: robot cirtesub, 9 links, 8 joints
Links:
- link cirtesub/base_link: geometry collision mesh filename=package://cirtesub_description/meshes/cirtesubdae_colisions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 scale=1 1 1; visual mesh filename=package://cirtesub_description/meshes/cirtesubdae.dae scale=1 1 1

File: urdf/cirtesub.urdf.xacro (robot description, xacro)
@@ -1,175 +1,287 @@
 <?xml version="1.0"?>
-<robot name="cirtesub" xmlns:xacro="http://ros.org/wiki/xacro">
-  <xacro:arg name="robot_namespace" default="cirtesub"/>
+<robot xmlns:xacro="http://www.ros.org/wiki/xacro" name="cirtesub" family="underwater">
+  <xacro:arg name="robot_name" default="cirtesub"/>
   <xacro:arg name="environment" default="sim"/>
   <xacro:arg name="lookup_csv" default="config/t200_lookup.csv"/>
   <xacro:arg name="stonefish_topic" default="/cirtesub/controller/thruster_setpoints_sim"/>
-  <xacro:arg name="pwm_channels" default="0,1,2,3,4,5,6,7"/>
   <xacro:arg name="pressure_offset_pa" default="101325.0"/>
-  <xacro:property name="robot_namespace" value="$(arg robot_namespace)"/>
-  <xacro:property name="robot_prefix" value="${robot_namespace}/"/>
-  <xacro:macro name="thruster_mount" params="link_name joint_name xyz rpy">
-    <link name="${link_name}"/>
-    <joint name="${joint_name}" type="fixed">
-      <parent link="${robot_prefix}base_link"/>
-      <child link="${link_name}"/>
-      <origin xyz="${xyz}" rpy="${rpy}"/>
-    </joint>
-  </xacro:macro>
-  <xacro:macro name="sensor_mount" params="link_name joint_name xyz rpy">
-    <link name="${link_name}"/>
-    <joint name="${joint_name}" type="fixed">
-      <parent link="${robot_prefix}base_link"/>
-      <child link="${link_name}"/>
-      <origin xyz="${xyz}" rpy="${rpy}"/>
-    </joint>
-  </xacro:macro>
-  <xacro:macro name="ros2_control_thruster_joint" params="joint_name">
-    <joint name="${joint_name}">
-      <command_interface name="effort"/>
-      <state_interface name="effort"/>
-    </joint>
-  </xacro:macro>
-  <xacro:macro name="ros2_control_sensor_system">
-    <ros2_control name="${robot_namespace}_sensors" type="system">
-      <hardware>
-        <plugin>sura_hardware_interface/SensorsSystem</plugin>
-        <param name="environment">$(arg environment)</param>
-        <param name="robot_namespace">${robot_namespace}</param>
-        <param name="sim_imu_topic">/${robot_namespace}/stonefish/sensors/imu</param>
-        <param name="sim_magnetometer_topic">/${robot_namespace}/stonefish/sensors/magnetometer</param>
-        <param name="sim_pressure_topic">/${robot_namespace}/stonefish/sensors/pressure</param>
-        <param name="sim_dvl_topic">/${robot_namespace}/stonefish/sensors/dvl</param>
-        <param name="sim_dvl_altitude_topic">/${robot_namespace}/stonefish/sensors/dvl/altitude</param>
-        <param name="sim_gps_topic">/${robot_namespace}/stonefish/sensors/gps</param>
-        <param name="pressure_offset_pa">$(arg pressure_offset_pa)</param>
-      </hardware>
-      <sensor name="imu_sensor">
-        <state_interface name="orientation.x"/>
-        <state_interface name="orientation.y"/>
-        <state_interface name="orientation.z"/>
-        <state_interface name="orientation.w"/>
-        <state_interface name="angular_velocity.x"/>
-        <state_interface name="angular_velocity.y"/>
-        <state_interface name="angular_velocity.z"/>
-        <state_interface name="linear_acceleration.x"/>
-        <state_interface name="linear_acceleration.y"/>
-        <state_interface name="linear_acceleration.z"/>
-      </sensor>
-      <sensor name="magnetometer_sensor">
-        <state_interface name="magnetic_field.x"/>
-        <state_interface name="magnetic_field.y"/>
-        <state_interface name="magnetic_field.z"/>
-      </sensor>
-      <sensor name="pressure_sensor">
-        <state_interface name="fluid_pressure"/>
-      </sensor>
-      <sensor name="battery_sensor">
-        <state_interface name="voltage"/>
-        <state_interface name="current"/>
-        <state_interface name="present"/>
-      </sensor>
-      <sensor name="dvl_sensor">
-        <state_interface name="linear_velocity.x"/>
-        <state_interface name="linear_velocity.y"/>
-        <state_interface name="linear_velocity.z"/>
-        <state_interface name="angular_velocity.x"/>
-        <state_interface name="angular_velocity.y"/>
-        <state_interface name="angular_velocity.z"/>
-        <state_interface name="distance_z"/>
-        <state_interface name="confidence"/>
-        <state_interface name="gps.latitude"/>
-        <state_interface name="gps.longitude"/>
-        <state_interface name="gps.altitude"/>
-        <state_interface name="gps.valid"/>
-      </sensor>
-    </ros2_control>
-  </xacro:macro>
-  <link name="${robot_prefix}base_link">
+  <!-- TF -->
+  <link name="$(arg robot_name)/base_link" tf_type="base">
     <visual>
       <origin xyz="0 0 0" rpy="0 -1.57 0"/>
       <geometry>
-        <mesh filename="package://cirtesub_description/meshes/cirtesubdae.dae" scale="1 1 1"/>
+        <mesh
+          filename="package://cirtesub_description/meshes/cirtesubdae.dae"
+          scale="1 1 1"/>
       </geometry>
     </visual>
+    <collision>
+      <origin xyz="0 0 0" rpy="0 -1.57 0"/>
+      <geometry>
+        <mesh
+          filename="package://cirtesub_description/meshes/cirtesubdae_colisions.dae"
+          scale="1 1 1"/>
+      </geometry>
+    </collision>
   </link>
-  <xacro:thruster_mount
-    link_name="${robot_prefix}Thruster_up_front"
-    joint_name="${robot_prefix}Thruster_up_front"
-    xyz="0.27 0.0 0.0"
-    rpy="1.57 1.57 0"/>
-  <xacro:thruster_mount
-    link_name="${robot_prefix}Thruster_up_back"
-    joint_name="${robot_prefix}Thruster_up_back"
-    xyz="-0.27 0.0 0.0"
-    rpy="1.57 1.57 0.0"/>
-  <xacro:thruster_mount
-    link_name="${robot_prefix}Thruster_up_left"
-    joint_name="${robot_prefix}Thruster_up_left"
-    xyz="0.0 -0.3 0.0"
-    rpy="1.57 1.57 0"/>
-  <xacro:thruster_mount
-    link_name="${robot_prefix}Thruster_up_right"
-    joint_name="${robot_prefix}Thruster_up_right"
-    xyz="0.0 0.30 0.0"
-    rpy="1.57 1.57 0"/>
-  <xacro:thruster_mount
-    link_name="${robot_prefix}Thruster_down_backleft"
-    joint_name="${robot_prefix}Thruster_down_backleft"
-    xyz="-0.165 -0.23 0.076"
-    rpy="0 0.0 2.35619"/>
-  <xacro:thruster_mount
-    link_name="${robot_prefix}Thruster_down_backright"
-    joint_name="${robot_prefix}Thruster_down_backright"
-    xyz="-0.165 0.23 0.076"
-    rpy="0 0.0 -2.35619"/>
-  <xacro:thruster_mount
-    link_name="${robot_prefix}Thruster_down_frontleft"
-    joint_name="${robot_prefix}Thruster_down_frontleft"
-    xyz="0.165 -0.23 0.076"
-    rpy="0 0.0 0.785398"/>
-  <xacro:thruster_mount
-    link_name="${robot_prefix}Thruster_down_frontright"
-    joint_name="${robot_prefix}Thruster_down_frontright"
-    xyz="0.165 0.23 0.076"
-    rpy="0 0.0 -0.7854"/>
-  <xacro:sensor_mount
-    link_name="${robot_prefix}IMU"
-    joint_name="${robot_prefix}IMU_joint"
-    xyz="0.0 0.0 0.0"
-    rpy="0.0 0.0 0.0"/>
-  <xacro:sensor_mount
-    link_name="${robot_prefix}Pressure"
-    joint_name="${robot_prefix}Pressure_joint"
-    xyz="0.0 0.0 -0.05"
-    rpy="0.0 0.0 0.0"/>
-  <xacro:sensor_mount
-    link_name="${robot_prefix}GPS"
-    joint_name="${robot_prefix}GPS_joint"
-    xyz="0.0 0.0 -0.40"
-    rpy="0.0 0.0 0.0"/>
-  <xacro:sensor_mount
-    link_name="${robot_prefix}DVL"
-    joint_name="${robot_prefix}DVL_joint"
-    xyz="0.0 0.0 0.15"
-    rpy="0.0 0.0 0.0"/>
-  <ros2_control name="${robot_namespace}_thrusters" type="system">
+  <!-- Sensors -->
+  <link name="$(arg robot_name)/imu_link" tf_type="sensor"/>
+  <joint name="$(arg robot_name)/imu_joint" type="fixed">
+    <parent link="$(arg robot_name)/base_link"/>
+    <child link="$(arg robot_name)/imu_link"/>
+    <origin xyz="0.0 0.0 0.0" rpy="0.0 0.0 0.0"/>
+  </joint>
+  <link name="$(arg robot_name)/pressure_link" tf_type="sensor"/>
+  <joint name="$(arg robot_name)/pressure_joint" type="fixed">
+    <parent link="$(arg robot_name)/base_link"/>
+    <child link="$(arg robot_name)/pressure_link"/>
+    <origin xyz="0.0 0.0 -0.05" rpy="0.0 0.0 0.0"/>
+  </joint>
+  <link name="$(arg robot_name)/GPS" tf_type="sensor"/>
+  <joint name="$(arg robot_name)/gps_joint" type="fixed">
+    <parent link="$(arg robot_name)/base_link"/>
+    <child link="$(arg robot_name)/GPS"/>
+    <origin xyz="0.0 0.0 -0.40" rpy="0.0 0.0 0.0"/>
+  </joint>
+  <link name="$(arg robot_name)/dvl_link" tf_type="sensor"/>
+  <joint name="$(arg robot_name)/dvl_joint" type="fixed">
+    <parent link="$(arg robot_name)/base_link"/>
+    <child link="$(arg robot_name)/dvl_link"/>
+    <origin xyz="0.0 0.0 0.15" rpy="0.0 0.0 0.0"/>
+  </joint>
+  <link name="$(arg robot_name)/down_camera/camera" tf_type="sensor"/>
+  <joint name="$(arg robot_name)/down_camera/camera_joint" type="fixed">
+    <parent link="$(arg robot_name)/base_link"/>
+    <child link="$(arg robot_name)/down_camera/camera"/>
+    <origin xyz="0.0 0.0 0.15" rpy="0.0 0.0 1.57"/>
+  </joint>
+  <link name="$(arg robot_name)/camera_down/optical_frame" tf_type="sensor"/>
+  <joint name="$(arg robot_name)/camera_down/optical_frame_joint" type="fixed">
+    <parent link="$(arg robot_name)/down_camera/camera"/>
+    <child link="$(arg robot_name)/camera_down/optical_frame"/>
+    <origin xyz="0.0 0.0 0.0" rpy="0.0 0.0 0.0"/>
+  </joint>
+  <!-- Thrusters -->
+  <link name="$(arg robot_name)/Thruster_up_front" tf_type="thruster"/>
+  <joint name="$(arg robot_name)/Thruster_up_front" type="fixed">
+    <parent link="$(arg robot_name)/base_link"/>
+    <child link="$(arg robot_name)/Thruster_up_front"/>
+    <origin xyz="0.27 0.0 0.0" rpy="1.57 1.57 0"/>
+  </joint>
+  <link name="$(arg robot_name)/Thruster_up_back" tf_type="thruster"/>
+  <joint name="$(arg robot_name)/Thruster_up_back" type="fixed">
+    <parent link="$(arg robot_name)/base_link"/>
+    <child link="$(arg robot_name)/Thruster_up_back"/>
+    <origin xyz="-0.27 0.0 0.0" rpy="1.57 1.57 0.0"/>
+  </joint>
+  <link name="$(arg robot_name)/Thruster_up_left" tf_type="thruster"/>
+  <joint name="$(arg robot_name)/Thruster_up_left" type="fixed">
+    <parent link="$(arg robot_name)/base_link"/>
+    <child link="$(arg robot_name)/Thruster_up_left"/>
+    <origin xyz="0.0 -0.3 0.0" rpy="1.57 1.57 0"/>
+  </joint>
+  <link name="$(arg robot_name)/Thruster_up_right" tf_type="thruster"/>
+  <joint name="$(arg robot_name)/Thruster_up_right" type="fixed">
+    <parent link="$(arg robot_name)/base_link"/>
+    <child link="$(arg robot_name)/Thruster_up_right"/>
+    <origin xyz="0.0 0.30 0.0" rpy="1.57 1.57 0"/>
+  </joint>
+  <link name="$(arg robot_name)/Thruster_down_backleft" tf_type="thruster"/>
+  <joint name="$(arg robot_name)/Thruster_down_backleft" type="fixed">
+    <parent link="$(arg robot_name)/base_link"/>
+    <child link="$(arg robot_name)/Thruster_down_backleft"/>
+    <origin xyz="-0.165 -0.23 0.076" rpy="0 0.0 2.35619"/>
+  </joint>
+  <link name="$(arg robot_name)/Thruster_down_backright" tf_type="thruster"/>
+  <joint name="$(arg robot_name)/Thruster_down_backright" type="fixed">
+    <parent link="$(arg robot_name)/base_link"/>
+    <child link="$(arg robot_name)/Thruster_down_backright"/>
+    <origin xyz="-0.165 0.23 0.076" rpy="0 0.0 -2.35619"/>
+  </joint>
+  <link name="$(arg robot_name)/Thruster_down_frontleft" tf_type="thruster"/>
+  <joint name="$(arg robot_name)/Thruster_down_frontleft" type="fixed">
+    <parent link="$(arg robot_name)/base_link"/>
+    <child link="$(arg robot_name)/Thruster_down_frontleft"/>
+    <origin xyz="0.165 -0.23 0.076" rpy="0 0.0 0.785398"/>
+  </joint>
+  <link name="$(arg robot_name)/Thruster_down_frontright" tf_type="thruster"/>
+  <joint name="$(arg robot_name)/Thruster_down_frontright" type="fixed">
+    <parent link="$(arg robot_name)/base_link"/>
+    <child link="$(arg robot_name)/Thruster_down_frontright"/>
+    <origin xyz="0.165 0.23 0.076" rpy="0 0.0 -0.7854"/>
+  </joint>
+  <!-- ROS2 CONTROL -->
+  <ros2_control name="$(arg robot_name)_thrusters" type="system">
     <hardware>
       <plugin>sura_hardware_interface/ThrustersSystem</plugin>
       <param name="environment">$(arg environment)</param>
-      <param name="lookup_csv">$(arg lookup_csv)</param>
-      <param name="stonefish_topic">$(arg stonefish_topic)</param>
-      <param name="pwm_channels">$(arg pwm_channels)</param>
     </hardware>
-    <!-- check the same order of the thrusters in stonefish -->
-    <xacro:ros2_control_thruster_joint joint_name="${robot_prefix}Thruster_up_front"/>
-    <xacro:ros2_control_thruster_joint joint_name="${robot_prefix}Thruster_up_back"/>
-    <xacro:ros2_control_thruster_joint joint_name="${robot_prefix}Thruster_up_left"/>
-    <xacro:ros2_control_thruster_joint joint_name="${robot_prefix}Thruster_up_right"/>
-    <xacro:ros2_control_thruster_joint joint_name="${robot_prefix}Thruster_down_backleft"/>
-    <xacro:ros2_control_thruster_joint joint_name="${robot_prefix}Thruster_down_backright"/>
-    <xacro:ros2_control_thruster_joint joint_name="${robot_prefix}Thruster_down_frontleft"/>
-    <xacro:ros2_control_thruster_joint joint_name="${robot_prefix}Thruster_down_frontright"/>
+    <joint name="$(arg robot_name)/Thruster_up_front">
+      <command_interface name="effort"/>
+      <state_interface name="effort"/>
+      <param name="lookup_csv">$(arg lookup_csv)</param>
+      <param name="stonefish_topic">$(arg stonefish_topic)</param>
+      <param name="inverted">false</param>
+      <param name="pwm_offset">0.0</param>
+      <param name="channel">0</param>
+      <param name="controller">thruster_test_controller</param>
+      <param name="controller">body_force</param>
+      <param name="controller">mpc_4dof</param>
+      <param name="controller">state_observer</param>
+      <param name="controller">body_velocity</param>
+      <param name="controller">position_hold</param>
+      <param name="controller">stabilize</param>
+      <param name="controller">depth_hold</param>
+    </joint>
+    <joint name="$(arg robot_name)/Thruster_up_back">
+      <command_interface name="effort"/>
+      <state_interface name="effort"/>
+      <param name="lookup_csv">$(arg lookup_csv)</param>
+      <param name="stonefish_topic">$(arg stonefish_topic)</param>
+      <param name="inverted">false</param>
+      <param name="pwm_offset">0.0</param>
+      <param name="channel">1</param>
+    </joint>
+    <joint name="$(arg robot_name)/Thruster_up_left">
+      <command_interface name="effort"/>
+      <state_interface name="effort"/>
+      <param name="lookup_csv">$(arg lookup_csv)</param>
+      <param name="stonefish_topic">$(arg stonefish_topic)</param>
+      <param name="inverted">false</param>
+      <param name="pwm_offset">0.0</param>
+      <param name="channel">2</param>
+    </joint>
+    <joint name="$(arg robot_name)/Thruster_up_right">
+      <command_interface name="effort"/>
+      <state_interface name="effort"/>
+      <param name="lookup_csv">$(arg lookup_csv)</param>
+      <param name="stonefish_topic">$(arg stonefish_topic)</param>
+      <param name="inverted">false</param>
+      <param name="pwm_offset">0.0</param>
+      <param name="channel">3</param>
+    </joint>
+    <joint name="$(arg robot_name)/Thruster_down_backleft">
+      <command_interface name="effort"/>
+      <state_interface name="effort"/>
+      <param name="lookup_csv">$(arg lookup_csv)</param>
+      <param name="stonefish_topic">$(arg stonefish_topic)</param>
+      <param name="inverted">false</param>
+      <param name="pwm_offset">0.0</param>
+      <param name="channel">4</param>
+    </joint>
+    <joint name="$(arg robot_name)/Thruster_down_backright">
+      <command_interface name="effort"/>
+      <state_interface name="effort"/>
+      <param name="lookup_csv">$(arg lookup_csv)</param>
+      <param name="stonefish_topic">$(arg stonefish_topic)</param>
+      <param name="inverted">false</param>
+      <param name="pwm_offset">0.0</param>
+      <param name="channel">5</param>
+    </joint>
+    <joint name="$(arg robot_name)/Thruster_down_frontleft">
+      <command_interface name="effort"/>
+      <state_interface name="effort"/>
+      <param name="lookup_csv">$(arg lookup_csv)</param>
+      <param name="stonefish_topic">$(arg stonefish_topic)</param>
+      <param name="inverted">false</param>
+      <param name="pwm_offset">0.0</param>
+      <param name="channel">6</param>
+    </joint>
+    <joint name="$(arg robot_name)/Thruster_down_frontright">
+      <command_interface name="effort"/>
+      <state_interface name="effort"/>
+      <param name="lookup_csv">$(arg lookup_csv)</param>
+      <param name="stonefish_topic">$(arg stonefish_topic)</param>
+      <param name="inverted">false</param>
+      <param name="pwm_offset">0.0</param>
+      <param name="channel">7</param>
+    </joint>
   </ros2_control>
-  <xacro:ros2_control_sensor_system/>
+  <ros2_control name="$(arg robot_name)_sensors" type="system">
+    <hardware>
+      <plugin>sura_hardware_interface/SensorsSystem</plugin>
+      <param name="environment">$(arg environment)</param>
+      <param name="robot_namespace">$(arg robot_name)</param>
+    </hardware>
+    <sensor name="imu_sensor">
+      <param name="interface">sura_hardware_interface/ImuInterface</param>
+      <param name="broadcaster">imu_broadcaster</param>
+      <param name="read_rate_hz">200.0</param>
+      <param name="frame_id">$(arg robot_name)/imu_link</param>
+      <param name="stonefish_topic">/$(arg robot_name)/stonefish/sensors/imu</param>
+      <param name="msg_type">sensor_msgs/msg/Imu</param>
+      <state_interface name="orientation.x"/>
+      <state_interface name="orientation.y"/>
+      <state_interface name="orientation.z"/>
+      <state_interface name="orientation.w"/>
+      <state_interface name="angular_velocity.x"/>
+      <state_interface name="angular_velocity.y"/>
+      <state_interface name="angular_velocity.z"/>
+      <state_interface name="linear_acceleration.x"/>
+      <state_interface name="linear_acceleration.y"/>
+      <state_interface name="linear_acceleration.z"/>
+      <state_interface name="sample_time.sec"/>
+      <state_interface name="sample_time.nanosec"/>
+    </sensor>
+    <sensor name="magnetometer_sensor">
+      <param name="interface">sura_hardware_interface/MagnetometerInterface</param>
+      <param name="broadcaster">magnetometer_broadcaster</param>
+      <param name="read_rate_hz">200.0</param>
+      <param name="frame_id">$(arg robot_name)/imu_link</param>
+      <param name="stonefish_topic">/$(arg robot_name)/stonefish/sensors/magnetometer</param>
+      <param name="msg_type">sensor_msgs/msg/MagneticField</param>
+      <state_interface name="magnetic_field.x"/>
+      <state_interface name="magnetic_field.y"/>
+      <state_interface name="magnetic_field.z"/>
+      <state_interface name="sample_time.sec"/>
+      <state_interface name="sample_time.nanosec"/>
+    </sensor>
+    <sensor name="pressure_sensor">
+      <param name="interface">sura_hardware_interface/PressureInterface</param>
+      <param name="broadcaster">pressure_broadcaster</param>
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