Commit message: added sensors frames

File: urdf/cirtesub_dual_alpha.urdf.xacro (robot description, xacro)
@@ -17,4 +17,12 @@
   <xacro:include filename="$(find alpha_description)/xacro/alpha.ros2_control.xacro"/>
   <xacro:macro name="thruster_mount" params="link_name joint_name xyz rpy">
+    <link name="${link_name}"/>
+    <joint name="${joint_name}" type="fixed">
+      <parent link="cirtesub/base_link"/>
+      <child link="${link_name}"/>
+      <origin xyz="${xyz}" rpy="${rpy}"/>
+    </joint>
+  </xacro:macro>
+  <xacro:macro name="sensor_mount" params="link_name joint_name xyz rpy">
     <link name="${link_name}"/>
     <joint name="${joint_name}" type="fixed">
@@ -78,4 +86,24 @@
     xyz="0.165 0.23 0.076"
     rpy="0 0.0 -0.7854"/>
+  <xacro:sensor_mount
+    link_name="cirtesub/IMU"
+    joint_name="cirtesub/IMU_joint"
+    xyz="0.0 0.0 0.0"
+    rpy="0.0 0.0 0.0"/>
+  <xacro:sensor_mount
+    link_name="cirtesub/Pressure"
+    joint_name="cirtesub/Pressure_joint"
+    xyz="0.0 0.0 -0.05"
+    rpy="0.0 0.0 0.0"/>
+  <xacro:sensor_mount
+    link_name="cirtesub/GPS"
+    joint_name="cirtesub/GPS_joint"
+    xyz="0.0 0.0 -0.40"
+    rpy="0.0 3.1416 0.0"/>
+  <xacro:sensor_mount
+    link_name="cirtesub/DVL"
+    joint_name="cirtesub/DVL_joint"
+    xyz="0.0 0.0 0.15"
+    rpy="0.0 0.0 0.0"/>
   <xacro:alpha_urdf
     parent="cirtesub/base_link"

Commit message: ajustes para agregar los yaml de ros2control

File: urdf/cirtesub_dual_alpha.urdf.xacro (robot description, xacro)
@@ -7,4 +7,5 @@
   <xacro:arg name="pwm_channels" default="0,1,2,3,4,5,6,7"/>
   <xacro:arg name="pressure_offset_pa" default="101325.0"/>
+  <xacro:arg name="arms" default="dual"/>
   <xacro:arg name="use_sim" default="true"/>
   <xacro:arg name="alpha_use_fake_hardware" default="true"/>
@@ -18,4 +19,5 @@
   <xacro:property name="robot_namespace" value="$(arg robot_namespace)"/>
   <xacro:property name="robot_prefix" value="${robot_namespace}/"/>
+  <xacro:property name="arms" value="$(arg arms)"/>
   <xacro:include filename="$(find alpha_description)/xacro/alpha.urdf.xacro"/>
   <xacro:include filename="$(find alpha_description)/xacro/alpha.ros2_control.xacro"/>
@@ -181,10 +183,12 @@
     <origin xyz="0.335 -0.165 0.145" rpy="-1.57 0.0 0.0"/>
   </xacro:alpha_urdf>
-  <xacro:alpha_urdf
-    parent="${robot_prefix}base_link"
-    prefix="${robot_prefix}alpha_right/"
-    description_package="alpha_description">
-    <origin xyz="0.335 0.165 0.145" rpy="1.57 0.0 0.0"/>
-  </xacro:alpha_urdf>
+  <xacro:if value="${arms == 'dual'}">
+    <xacro:alpha_urdf
+      parent="${robot_prefix}base_link"
+      prefix="${robot_prefix}alpha_right/"
+      description_package="alpha_description">
+      <origin xyz="0.335 0.165 0.145" rpy="1.57 0.0 0.0"/>
+    </xacro:alpha_urdf>
+  </xacro:if>
   <ros2_control name="${robot_namespace}_thrusters" type="system">
     <hardware>
@@ -217,14 +221,16 @@
     use_sim="$(arg use_sim)"
     use_fake_hardware="$(arg alpha_use_fake_hardware)"/>
-  <xacro:alpha_system
-    prefix="${robot_prefix}alpha_right/"
-    name="${robot_prefix}alpha_right"
-    serial_port="$(arg alpha_right_serial_port)"
-    state_update_frequency="$(arg alpha_right_state_update_frequency)"
-    initial_positions_file="$(arg initial_positions_file)"
-    description_package="alpha_description"
-    desired_joint_states_topic="$(arg alpha_desired_joint_states_topic)"
-    joint_states_topic="$(arg alpha_joint_states_topic)"
-    use_sim="$(arg use_sim)"
-    use_fake_hardware="$(arg alpha_use_fake_hardware)"/>
+  <xacro:if value="${arms == 'dual'}">
+    <xacro:alpha_system
+      prefix="${robot_prefix}alpha_right/"
+      name="${robot_prefix}alpha_right"
+      serial_port="$(arg alpha_right_serial_port)"
+      state_update_frequency="$(arg alpha_right_state_update_frequency)"
+      initial_positions_file="$(arg initial_positions_file)"
+      description_package="alpha_description"
+      desired_joint_states_topic="$(arg alpha_desired_joint_states_topic)"
+      joint_states_topic="$(arg alpha_joint_states_topic)"
+      use_sim="$(arg use_sim)"
+      use_fake_hardware="$(arg alpha_use_fake_hardware)"/>
+  </xacro:if>
 </robot>

Commit message: change the rotation of the arms

File: urdf/cirtesub_dual_alpha.urdf.xacro (robot description, xacro)
@@ -15,5 +15,6 @@
   <xacro:arg name="initial_positions_file" default="initial_positions.yaml"/>
   <xacro:arg name="alpha_desired_joint_states_topic" default="/cirtesub/alpha/desired_joint_states"/>
-  <xacro:arg name="alpha_joint_states_topic" default="/cirtesub/alpha/joint_states"/>
+  <xacro:arg name="alpha_joint_states_topic" default="/cirtesub/stonefish/alpha/joint_states"/>
+  <xacro:arg name="alpha_normalized_joint_states_topic" default="/cirtesub/alpha/joint_states"/>
   <xacro:property name="arms" value="$(arg arms)"/>
   <xacro:include filename="$(find alpha_description)/xacro/alpha.urdf.xacro"/>
@@ -135,5 +136,5 @@
     prefix="$(arg robot_name)/alpha_left/"
     description_package="alpha_description">
-    <origin xyz="0.335 -0.165 0.145" rpy="-1.57 0.0 0.0"/>
+    <origin xyz="0.335 -0.165 0.145" rpy="0.0 0.0 0.0"/>
   </xacro:alpha_urdf>
   <xacro:if value="${arms == 'dual'}">
@@ -142,5 +143,5 @@
       prefix="$(arg robot_name)/alpha_right/"
       description_package="alpha_description">
-      <origin xyz="0.335 0.165 0.145" rpy="1.57 0.0 0.0"/>
+      <origin xyz="0.335 0.165 0.145" rpy="0.0 0.0 0.0"/>
     </xacro:alpha_urdf>
   </xacro:if>
@@ -330,4 +331,5 @@
     desired_joint_states_topic="$(arg alpha_desired_joint_states_topic)"
     joint_states_topic="$(arg alpha_joint_states_topic)"
+    normalized_joint_states_topic="$(arg alpha_normalized_joint_states_topic)"
     use_sim="$(arg use_sim)"
     use_fake_hardware="$(arg alpha_use_fake_hardware)"/>
@@ -342,4 +344,5 @@
       desired_joint_states_topic="$(arg alpha_desired_joint_states_topic)"
       joint_states_topic="$(arg alpha_joint_states_topic)"
+      normalized_joint_states_topic="$(arg alpha_normalized_joint_states_topic)"
       use_sim="$(arg use_sim)"
       use_fake_hardware="$(arg alpha_use_fake_hardware)"/>
