Commit message: robot con payload

File: moveit2/cirtesub_dual_alpha.srdf.xacro (robot description, xacro)
@@ -2,5 +2,18 @@
 <robot name="cirtesub" xmlns:xacro="http://www.ros.org/wiki/xacro">
   <xacro:arg name="robot_name" default="cirtesub"/>
+  <xacro:arg name="floating_base" default="false"/>
+  <xacro:arg name="world_frame" default="world_ned"/>
   <xacro:property name="robot" value="$(arg robot_name)"/>
+  <xacro:if value="$(arg floating_base)">
+    <virtual_joint name="world_joint" type="floating" parent_frame="$(arg world_frame)" child_link="${robot}/base_link"/>
+    <group name="base_alpha_left">
+      <joint name="world_joint"/>
+      <group name="alpha_left"/>
+    </group>
+    <group name="base_alpha_right">
+      <joint name="world_joint"/>
+      <group name="alpha_right"/>
+    </group>
+  </xacro:if>
   <group name="alpha_left">
     <link name="${robot}/alpha_left/ee_base_link"/>

File: urdf/cirtesub_dual_alpha.urdf.xacro (robot description, xacro)
@@ -23,13 +23,13 @@
   <link name="$(arg robot_name)/base_link" tf_type="base">
     <visual>
-      <origin xyz="0 0 0" rpy="0 -1.57 0"/>
+      <origin xyz="0 0 0" rpy="0 3.1416 1.57"/>
       <geometry>
         <mesh
-          filename="package://cirtesub_description/meshes/cirtesubdae.dae"
+          filename="package://cirtesub_description/meshes/cirtesub_v2_alpha.dae"
           scale="1 1 1"/>
       </geometry>
     </visual>
     <collision>
-      <origin xyz="0 0 0" rpy="0 -1.57 0"/>
+      <origin xyz="0 0 0" rpy="0 3.1416 1.57"/>
       <geometry>
         <mesh
@@ -136,5 +136,5 @@
     prefix="$(arg robot_name)/alpha_left/"
     description_package="alpha_description">
-    <origin xyz="0.335 -0.165 0.145" rpy="0.0 0.0 0.0"/>
+    <origin xyz="0.2664 -0.2090 0.0322" rpy="0.0 0.0 0.0"/>
   </xacro:alpha_urdf>
   <xacro:if value="${arms == 'dual'}">
@@ -143,5 +143,5 @@
       prefix="$(arg robot_name)/alpha_right/"
       description_package="alpha_description">
-      <origin xyz="0.335 0.165 0.145" rpy="0.0 0.0 0.0"/>
+      <origin xyz="0.2664 0.2136 0.0322" rpy="0.0 0.0 0.0"/>
     </xacro:alpha_urdf>
   </xacro:if>
